Commit message: Agregando error con la ruta de los motores.

File: models/rov_version1/urdf/rov_snippets.xacro (robot description, xacro)
@@ -4,5 +4,5 @@
   over propeller's frame X-axis in DAE (Collada) or STL format.
   -->
-  <xacro:property name="prop_mesh_file" value="file://$(find robocol_rov)/mesh/robocol_rov_motores.dae"/>
+  <xacro:property name="prop_mesh_file" value="file://$(find robocol_rov)/models/rov_version1/mesh/robocol_rov_motores.dae"/>
   <!-- Thruster macro with integration of joint and link-->
   <xacro:macro name="thruster_macro" params="robot_namespace thruster_id *origin">

Commit message: Arreglando cosas

File: models/rov_version1/urdf/rov_snippets.xacro (robot description, xacro)
@@ -47,5 +47,5 @@
         <gain>1</gain>
         <!-- Maximum allowed input value for the input signal for thruster unit -->
-        <clampMax>0</clampMax>
+        <clampMax>0</clampMax> <!-- Mirar las restricciones del motor -->
         <!-- Minimum allowed value for the input signal for thruster unit -->
         <clampMin>0</clampMin>

File: models/rov_version1/urdf/rov_thrusters.xacro (robot description, xacro)
@@ -5,6 +5,7 @@
     robot_namespace="${namespace}"
     thruster_id="0">
-    <origin xyz="0 0 0" rpy="0 0 ${pi}" />
+    <origin xyz="0.2 0.2 0.2" rpy="0 0 ${pi}" />
   </xacro:thruster_macro>
+<!--
   <xacro:thruster_macro
     robot_namespace="${namespace}"
@@ -17,3 +18,19 @@
     <origin xyz="0 0 0" rpy="0 -${0.5*pi} 0" />
   </xacro:thruster_macro>
+  <xacro:thruster_macro
+    robot_namespace="${namespace}"
+    thruster_id="3">
+    <origin xyz="0 0 0" rpy="pi 0 ${pi}" />
+  </xacro:thruster_macro>
+  <xacro:thruster_macro
+    robot_namespace="${namespace}"
+    thruster_id="4">
+    <origin xyz="0 0 0" rpy="-pi/2 0 ${pi}" />
+  </xacro:thruster_macro>
+  <xacro:thruster_macro
+    robot_namespace="${namespace}"
+    thruster_id="5">
+    <origin xyz="0 0 0" rpy="pi/2 -${0.5*pi} 0" />
+  </xacro:thruster_macro>
+-->
 </robot>
