Commit message: Arreglando errores

File: models/rov_version1/robots/rov_version1.xacro (robot description, xacro)
@@ -11,5 +11,5 @@
   <!-- Joint state publisher plugin -->
   <gazebo>
-    <plugin name="joint_state_publisher" filename="libjoint_state_publisher.so">
+    <plugin name="joint_state_publisher" filename="libuuv_joint_state_publisher.so">
       <robotNamespace>$(arg namespace)</robotNamespace>
       <updateRate>50</updateRate>

File: models/rov_version1/urdf/rov_base.xacro (robot description, xacro)
@@ -89,6 +89,6 @@
   </joint>
     <!-- Set up hydrodynamic plugin -->
-    <gazebo>
-      <plugin name="${namespace}_uuv_plugin" filename="libunderwater_object_ros_plugin.so">
+    <gazebo><!--  -->
+      <plugin name="${namespace}_uuv_plugin" filename="libuuv_underwater_object_ros_plugin.so">
         <!-- Fluid density to be used in the computation of buoyancy forces
         for all links specified below -->
@@ -125,10 +125,10 @@
             <type>fossen</type>
             <added_mass>
-              0 0 0 0 0 0
-              0 0 0 0 0 0
-              0 0 0 0 0 0
-              0 0 0 0 0 0
-              0 0 0 0 0 0
-              0 0 0 0 0 0
+                     779.79 -6.8773 -103.32  8.5426 -165.54 -7.8033
+                    -6.8773    1222   51.29  409.44 -5.8488  62.726
+                    -103.32   51.29  3659.9  6.1112 -386.42  10.774
+                     8.5426  409.44  6.1112   534.9 -10.027  21.019
+                    -165.54 -5.8488 -386.42 -10.027  842.69 -1.1162
+                    -7.8033  62.726  10.775  21.019 -1.1162  224.32
             </added_mass>
             <!--
@@ -137,5 +137,5 @@
             -->
             <linear_damping>
-              0 0 0 0 0 0
+              -74.82 -69.48 -728.4 -268.8 -309.77 -105
             </linear_damping>
             <!--
@@ -146,5 +146,6 @@
             -->
             <linear_damping_forward_speed>
-              0 0 0 0 0 0
+		0 0 0 0 0 0
+              <!---74.82 -69.48 -728.4 -268.8 -309.77 -105 -->
             </linear_damping_forward_speed>
             <!--
@@ -153,5 +154,5 @@
             -->
             <quadratic_damping>
-              0 0 0 0 0 0
+              -748.22 -992.53 -1821.01 -672 -774.44 -523.27
             </quadratic_damping>
           </hydrodynamic_model>

File: models/rov_version1/urdf/rov_snippets.xacro (robot description, xacro)
@@ -40,4 +40,5 @@
         <!-- Name of the joint between thruster and vehicle base link -->
         <jointName>${robot_namespace}/thruster_${thruster_id}_joint</jointName>
+	<thrusterID>${thruster_id}</thrusterID>
         <!-- Thruster force output topic name -->
         <thrustTopic>${robot_namespace}/thrusters/${thruster_id}/thrust</thrustTopic>
@@ -47,7 +48,7 @@
         <gain>1</gain>
         <!-- Maximum allowed input value for the input signal for thruster unit -->
-        <clampMax>0</clampMax> <!-- Mirar las restricciones del motor -->
+        <clampMax>2000</clampMax> <!-- Mirar las restricciones del motor -->
         <!-- Minimum allowed value for the input signal for thruster unit -->
-        <clampMin>0</clampMin>
+        <clampMin>1000</clampMin>
         <!--
         Value from 0 to 1 to set the efficiency of the output thrust force

File: models/rov_version1/urdf/rov_thrusters.xacro (robot description, xacro)
@@ -2,4 +2,5 @@
 <robot xmlns:xacro="http://www.ros.org/wiki/xacro">
   <!-- Adding the thruster units with the macro created in rov_example_snippets.xacro -->
+  <!--
   <xacro:thruster_macro
     robot_namespace="${namespace}"
@@ -7,30 +8,4 @@
     <origin xyz="0.2 0.2 0.2" rpy="0 0 ${pi}" />
   </xacro:thruster_macro>
-<!--
-  <xacro:thruster_macro
-    robot_namespace="${namespace}"
-    thruster_id="1">
-    <origin xyz="0 0 0" rpy="0 0 ${pi}" />
-  </xacro:thruster_macro>
-  <xacro:thruster_macro
-    robot_namespace="${namespace}"
-    thruster_id="2">
-    <origin xyz="0 0 0" rpy="0 -${0.5*pi} 0" />
-  </xacro:thruster_macro>
-  <xacro:thruster_macro
-    robot_namespace="${namespace}"
-    thruster_id="3">
-    <origin xyz="0 0 0" rpy="pi 0 ${pi}" />
-  </xacro:thruster_macro>
-  <xacro:thruster_macro
-    robot_namespace="${namespace}"
-    thruster_id="4">
-    <origin xyz="0 0 0" rpy="-pi/2 0 ${pi}" />
-  </xacro:thruster_macro>
-  <xacro:thruster_macro
-    robot_namespace="${namespace}"
-    thruster_id="5">
-    <origin xyz="0 0 0" rpy="pi/2 -${0.5*pi} 0" />
-  </xacro:thruster_macro>
--->
+  -->
 </robot>
